File: HARDWARE/verdaderamente el proyecto - copia/nahue.kicad_sch (KiCad schematic)
At the start: 38 parts, among them J2 Screw_Terminal_01x03, J3 Screw_Terminal_01x03, J4 Screw_Terminal_01x03, J5 bateria, J6 Screw_Terminal_01x03, K1 JQC-3FF-005-1Z, K2 JQC-3FF-005-1Z, K3 JQC-3FF-005-1Z, K4 JQC-3FF-005-1Z, Q1 BC847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

Commit message: actualizacion del kicad
Parts:
- added C1, C2: C_Small, Capacitor_THT:C_Axial_L5.1mm_D3.1mm_P10.00mm_Horizontal, symbol Device:C_Small
- added J1, J7: Conn_01x15, Connector_PinHeader_2.54mm:PinHeader_1x15_P2.54mm_Vertical, symbol Connector_Generic:Conn_01x15
- Q1, Q2, Q3, Q4: value BC847 -> MMBT3904
- R1, R10, R4, R7: value 220k -> 220
Connections:
- net vinESP is gone; now on net +5V: U5.3 (VO)
- net +5V: now also C1.1, C2.1, J1.15 (Pin_15)
- net GND: now also C1.2, C2.2, J1.14 (Pin_14), J7.2 (Pin_2)
- net NC1: no longer J3.3 (Pin_3), K1.11
- net INPUT1 renamed D21
- net D21: now also J7.11 (Pin_11)
- net INPUT2 renamed D19
- net D19: now also J7.10 (Pin_10)
- net INPUT3 renamed D18
- net D18: now also J7.9 (Pin_9)
- net INPUT4 renamed D5
- net D5: now also J7.8 (Pin_8)
- new net 3V3: J7.1 (Pin_1)
- new net COM1: J3.3 (Pin_3), K1.11
- new net D12: J1.12 (Pin_12)
- new net D13: J1.13 (Pin_13)
- new net D14: J1.11 (Pin_11)
- new net D15: J7.3 (Pin_3)
- new net D2: J7.4 (Pin_4)
- new net D22: J7.14 (Pin_14)
- new net D23: J7.15 (Pin_15)
- new net D25: J1.8 (Pin_8)
- new net D26: J1.9 (Pin_9)
- new net D27: J1.10 (Pin_10)
- new net D32: J1.6 (Pin_6)
- new net D33: J1.7 (Pin_7)
- new net D34: J1.4 (Pin_4)
- new net D35: J1.5 (Pin_5)
- new net D4: J7.5 (Pin_5)
- new net DX2: J7.7 (Pin_7)
- new net EN: J1.1 (Pin_1)
- new net RX0: J7.12 (Pin_12)
- new net RX2: J7.6 (Pin_6)
- new net TX0: J7.13 (Pin_13)
- new net VN: J1.3 (Pin_3)
- new net VP: J1.2 (Pin_2)
Other:
- moved on the sheet: J5, U5
