File: HARDWARE/nahue.kicad_pcb (KiCad board)
At the start: 2 copper layers, 97.2 x 86.4 mm, 86 parts, among them J2 Screw_Terminal_01x03, J4 Screw_Terminal_01x03, J5 Screw_Terminal_01x03, J6 Conn_01x08, K1 RELAY, K2 RELAY, K3 RELAY, K4 RELAY, Q1 MMBT3904, Q2 MMBT3904, Q3 MMBT3904, Q4 MMBT3904, SW1 SW, U1 PC817, U2 PC817, U3 PC817, U4 PC817, U6 LM7805_TO220

Commit message: duplicacion de placa
Parts:
- moved J2 13.1 mm to (179.3, 79.1)
- moved J3 13.1 mm to (179.3, 98.0)
- moved J4 13.1 mm to (179.3, 135.7)
- moved J5 13.1 mm to (179.3, 117.0)
- moved K1 13.1 mm to (202.6, 80.1)
- moved K2 13.1 mm to (202.4, 99.1)
- moved K3 13.1 mm to (202.4, 136.7)
- moved K4 13.1 mm to (202.4, 118.1)
- moved R1 13.1 mm to (236.4, 123.8)
- moved R11 13.1 mm to (220.3, 75.5)
- moved R2 13.1 mm to (220.7, 132.3)
- moved R5 13.1 mm to (220.7, 113.5)
- moved R8 13.1 mm to (220.3, 94.5)
- moved SW1 13.1 mm to (264.4, 125.5)
- moved U1 13.1 mm to (231.3, 72.9)
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Routing:
- removed copper zone on B.Cu, net (none)
Other:
- board outline removed

Commit message: imprimir placa
Parts:
- removed C1 (x2): ~, Capacitor_THT:C_Axial_L5.1mm_D3.1mm_P10.00mm_Horizontal
- removed C2 (x2): ~, Capacitor_THT:CP_Radial_D8.0mm_P3.80mm
- removed the D1 at (88.2, 128.4)
- removed the D1 at (220.3, 128.5)
- removed the D2 at (209.4, 130.9)
- removed the D2 at (77.3, 130.8)
- removed the D3 at (88.7, 109.7)
- removed the D3 at (220.8, 109.7)
- removed the D4 at (209.4, 112.1)
- removed the D4 at (77.3, 112.0)
- removed the D5 at (88.2, 90.7)
- removed the D5 at (220.3, 90.7)
- removed the D6 at (209.4, 93.1)
- removed the D6 at (77.3, 93.0)
- removed the D7 at (87.7, 71.6)
- removed the D7 at (219.8, 71.7)
- removed the D8 at (209.4, 74.1)
- removed the D8 at (77.3, 74.0)
- removed J1 (x2): ~, TerminalBlock:TerminalBlock_MaiXu_MX126-5.0-02P_1x02_P5.00mm
- removed J2 (x2), J4 (x2), J5 (x2): Screw_Terminal_01x03, TerminalBlock:TerminalBlock_MaiXu_MX126-5.0-03P_1x03_P5.00mm
- removed J3 (x2): ~, TerminalBlock:TerminalBlock_MaiXu_MX126-5.0-03P_1x03_P5.00mm
- removed J6 (x2): Conn_01x08, Connector_PinSocket_2.54mm:PinSocket_1x08_P2.54mm_Vertical
- removed K1 (x2), K2 (x2), K3 (x2), K4 (x2): RELAY, Relay_THT:Relay_SPDT_Hongfa_JQC-3FF_0XX-1Z
- removed the Q1 at (214.8, 76.5)
- removed the Q1 at (82.7, 76.4)
- removed the Q2 at (82.7, 95.4)
- removed the Q2 at (214.8, 95.5)
- removed the Q3 at (82.7, 133.2)
- removed the Q3 at (214.8, 133.3)
- removed the Q4 at (214.8, 114.5)
- removed the Q4 at (82.7, 114.4)
- removed the R1 at (104.3, 123.7)
- removed the R1 at (236.4, 123.8)
- removed the R10 at (102.4, 68.3)
- removed the R10 at (234.5, 68.3)
- removed the R11 at (88.2, 75.5)
- removed the R11 at (220.3, 75.5)
- removed the R12 at (82.7, 71.6)
- removed the R12 at (214.8, 71.7)
- removed the R2 at (88.6, 132.3)
- removed the R2 at (220.7, 132.3)
- removed the R3 at (214.8, 128.5)
- removed the R3 at (82.7, 128.4)
- removed the R4 at (235.7, 105.4)
- removed the R4 at (103.5, 105.3)
- removed the R5 at (220.7, 113.5)
- removed the R5 at (88.6, 113.5)
- removed the R6 at (82.7, 109.6)
- removed the R6 at (214.8, 109.7)
- removed the R7 at (235.5, 86.4)
- removed the R7 at (103.4, 86.3)
- removed the R8 at (220.3, 94.5)
- removed the R8 at (88.2, 94.4)
- removed the R9 at (214.8, 90.7)
- removed the R9 at (82.7, 90.7)
- removed SW1 (x2): SW, Connector_PinHeader_2.54mm:PinHeader_1x02_P2.54mm_Vertical
- removed the U1 at (231.3, 72.9)
- removed the U1 at (99.2, 72.9)
- removed the U2 at (99.2, 91.9)
- removed the U2 at (231.3, 92.0)
- removed the U3 at (232.2, 129.8)
- removed the U3 at (100.0, 129.7)
- removed the U4 at (99.3, 110.9)
- removed the U4 at (231.4, 111.0)
- removed U5 (x2): ~, esp32-30pines:esp32
- removed U6 (x2): LM7805_TO220, Package_TO_SOT_THT:TO-220-3_Vertical
- added ?: , , F.Cu at (172.0, 77.6)
- added ?: , , F.Cu at (122.5, 38.5)
- added ?: , , F.Cu at (247.8, 132.8)
- added ?: , , F.Cu at (122.7, 151.5)
- added ?: , , F.Cu at (60.1, 87.1)
- added ?: , , F.Cu at (113.3, 66.0)
- added ?: , , F.Cu at (259.5, 105.9)
- added ?: , , F.Cu at (172.0, 134.2)
- added ?: , , F.Cu at (182.9, 102.6)
- added ?: , , F.Cu at (97.2, 121.0)
- added ?: , , F.Cu at (183.1, 71.6)
- added ?: , , F.Cu at (46.2, 129.2)
- added ?: , , F.Cu at (46.0, 136.2)
- added ?: , , F.Cu at (195.1, 128.2)
- added ?: , , F.Cu at (254.6, 129.0)
- added ?: , , F.Cu at (35.1, 123.2)
- added ?: , , F.Cu at (97.0, 58.8)
- added ?: , , F.Cu at (97.0, 25.8)
- added ?: , , F.Cu at (234.0, 88.1)
- added ?: , , F.Cu at (197.1, 115.6)
- added ?: , , F.Cu at (97.0, 38.5)
- added ?: , , F.Cu at (60.4, 123.2)
- added ?: , , F.Cu at (195.1, 140.2)
- added ?: , , F.Cu at (105.8, 158.7)
- added ?: , , F.Cu at (35.0, 73.4)
- added ?: , , F.Cu at (35.1, 161.1)
- added ?: , , F.Cu at (105.7, 66.0)
- added ?: , , F.Cu at (195.1, 90.6)
- added ?: , , F.Cu at (122.5, 56.2)
- added ?: , , F.Cu at (97.2, 115.9)
- added ?: , , F.Cu at (118.4, 66.0)
- added ?: , , F.Cu at (35.1, 179.8)
- added ?: , , F.Cu at (195.3, 83.6)
- added ?: , , F.Cu at (58.1, 43.5)
- added ?: , , F.Cu at (247.8, 142.0)
- added ?: , , F.Cu at (46.0, 148.2)
- added ?: , , F.Cu at (110.9, 158.7)
- added ?: , , F.Cu at (172.0, 139.2)
- added ?: , , F.Cu at (197.3, 77.6)
- added ?: , , F.Cu at (259.5, 75.4)
- added ?: , , F.Cu at (35.1, 184.8)
- added ?: , , F.Cu at (35.1, 147.1)
- added ?: , , F.Cu at (250.3, 113.1)
- added ?: , , F.Cu at (108.5, 187.6)
- added ?: , , F.Cu at (122.5, 58.8)
- added ?: , , F.Cu at (172.0, 101.5)
- added ?: , , F.Cu at (122.7, 141.3)
- added ?: , , F.Cu at (122.5, 53.7)
- added ?: , , F.Cu at (195.3, 71.6)
- added ?: , , F.Cu at (97.2, 143.9)
- added ?: , , F.Cu at (35.0, 49.4)
- added ?: , , F.Cu at (259.5, 72.9)
- added ?: , , F.Cu at (234.0, 105.9)
- added ?: , , F.Cu at (234.0, 85.6)
- added ?: , , F.Cu at (120.2, 81.9)
- added ?: , , F.Cu at (97.0, 28.3)
- added ?: , , F.Cu at (58.1, 74.5)
- added ?: , , F.Cu at (97.0, 23.2)
- added ?: , , F.Cu at (122.5, 51.2)
- added ?: , , F.Cu at (259.5, 80.5)
- added ?: , , F.Cu at (35.1, 174.8)
- added ?: , , F.Cu at (259.5, 93.2)
- added ?: , , F.Cu at (35.1, 137.1)
- added ?: , , F.Cu at (122.7, 126.1)
- added ?: , , F.Cu at (120.2, 187.6)
- added ?: , , F.Cu at (110.8, 66.0)
- added ?: , , F.Cu at (195.1, 121.6)
- added ?: , , F.Cu at (182.9, 90.6)
- added ?: , , F.Cu at (60.2, 179.8)
- added ?: , , F.Cu at (122.5, 43.5)
- added ?: , , F.Cu at (58.2, 185.8)
- added ?: , , F.Cu at (182.9, 140.2)
- added ?: , , F.Cu at (58.1, 62.5)
- added ?: , , F.Cu at (58.1, 93.1)
- added ?: , , F.Cu at (97.0, 46.1)
- added ?: , , F.Cu at (35.0, 92.1)
- added ?: , , F.Cu at (259.5, 85.6)
- added ?: , , F.Cu at (122.5, 25.8)
- added ?: , , F.Cu at (259.5, 78.0)
- added ?: , , F.Cu at (105.9, 187.6)
- added ?: , , F.Cu at (252.8, 113.1)
- added ?: , , F.Cu at (45.9, 43.5)
- added ?: , , F.Cu at (122.5, 46.1)
- added ?: , , F.Cu at (35.1, 166.1)
- added ?: , , F.Cu at (58.4, 129.2)
- added ?: , , F.Cu at (97.2, 148.9)
- added ?: , , F.Cu at (122.7, 146.4)
- added ?: , , F.Cu at (97.2, 146.4)
- added ?: , , F.Cu at (122.5, 33.4)
- added ?: , , F.Cu at (46.0, 173.8)
- added ?: , , F.Cu at (172.0, 120.5)
- added ?: , , F.Cu at (182.9, 121.6)
- added ?: , , F.Cu at (247.7, 113.1)
- added ?: , , F.Cu at (257.1, 142.0)
- added ?: , , F.Cu at (60.2, 161.2)
- added ?: , , F.Cu at (234.0, 75.4)
- added ?: , , F.Cu at (100.7, 158.7)
- added ?: , , F.Cu at (259.5, 100.8)
- added ?: , , F.Cu at (110.9, 85.7)
- added ?: , , F.Cu at (60.2, 142.2)
- added ?: , , F.Cu at (122.7, 143.9)
- added ?: , , F.Cu at (257.1, 137.0)
- added ?: , , F.Cu at (35.0, 87.1)
- added ?: , , F.Cu at (97.2, 136.2)
- added ?: , , F.Cu at (245.3, 142.0)
- added ?: , , F.Cu at (120.2, 182.6)
- added ?: , , F.Cu at (97.0, 35.9)
- added ?: , , F.Cu at (97.2, 141.3)
- added ?: , , F.Cu at (122.5, 35.9)
- added ?: , , F.Cu at (120.2, 174.6)
- added ?: , , F.Cu at (97.0, 181.6)
- added ?: , , F.Cu at (58.2, 155.2)
- added ?: , , F.Cu at (122.7, 136.2)
- added ?: , , F.Cu at (35.0, 25.5)
- added ?: , , F.Cu at (172.0, 82.6)
- added ?: , , F.Cu at (122.7, 148.9)
- added ?: , , F.Cu at (97.0, 43.5)
- added ?: , , F.Cu at (122.7, 118.5)
- added ?: , , F.Cu at (115.9, 66.0)
- added ?: , , F.Cu at (172.0, 129.2)
- added ?: , , F.Cu at (111.0, 178.3)
- added ?: , , F.Cu at (35.0, 68.4)
- added ?: , , F.Cu at (110.9, 75.7)
- added ?: , , F.Cu at (97.2, 128.6)
- added ?: , , F.Cu at (35.0, 54.4)
- added ?: , , F.Cu at (120.1, 89.9)
- added ?: , , F.Cu at (35.0, 82.1)
- added ?: , , F.Cu at (96.9, 88.9)
- added ?: , , F.Cu at (108.2, 66.0)
- added ?: , , F.Cu at (172.0, 96.5)
- added ?: , , F.Cu at (257.1, 129.0)
- added ?: , , F.Cu at (247.8, 122.8)
- added ?: , , F.Cu at (100.8, 181.6)
- added ?: , , F.Cu at (242.8, 142.0)
- added ?: , , F.Cu at (58.3, 24.5)
- added ?: , , F.Cu at (58.3, 36.5)
- added ?: , , F.Cu at (234.0, 90.7)
- added ?: , , F.Cu at (97.0, 41.0)
- added ?: , , F.Cu at (110.9, 94.9)
- added ?: , , F.Cu at (122.5, 30.8)
- added ?: , , F.Cu at (234.0, 83.0)
- added ?: , , F.Cu at (172.0, 115.5)
- added ?: , , F.Cu at (122.7, 128.6)
- added ?: , , F.Cu at (45.9, 81.1)
- added ?: , , F.Cu at (35.1, 156.1)
- added ?: , , F.Cu at (97.2, 131.2)
- added ?: , , F.Cu at (45.9, 93.1)
- added ?: , , F.Cu at (116.0, 158.7)
- added ?: , , F.Cu at (234.0, 103.4)
- added ?: , , F.Cu at (97.0, 51.2)
- added ?: , , F.Cu at (122.5, 28.3)
- added ?: , , F.Cu at (58.1, 81.1)
- added ?: , , F.Cu at (97.0, 30.8)
- added ?: , , F.Cu at (97.0, 53.7)
- added ?: , , F.Cu at (58.2, 148.2)
- added ?: , , F.Cu at (240.1, 113.1)
- added ?: , , F.Cu at (100.6, 66.0)
- added ?: , , F.Cu at (195.1, 102.6)
- added ?: , , F.Cu at (108.3, 158.7)
- added ?: , , F.Cu at (234.0, 93.2)
- added ?: , , F.Cu at (259.5, 70.3)
- added ?: , , F.Cu at (46.1, 36.5)
- added ?: , , F.Cu at (97.0, 56.2)
- added ?: , , F.Cu at (46.1, 24.5)
- added ?: , , F.Cu at (234.0, 95.7)
- added ?: , , F.Cu at (97.2, 118.5)
- added ?: , , F.Cu at (234.0, 78.0)
- added ?: , , F.Cu at (259.5, 95.7)
- added ?: , , F.Cu at (259.5, 103.4)
- added ?: , , F.Cu at (237.7, 136.0)
- added ?: , , F.Cu at (259.5, 98.3)
- added ?: , , F.Cu at (234.0, 72.9)
- added ?: , , F.Cu at (120.1, 94.9)
- added ?: , , F.Cu at (245.2, 113.1)
- added ?: , , F.Cu at (35.1, 128.2)
- added ?: , , F.Cu at (234.0, 80.5)
- added ?: , , F.Cu at (103.3, 158.7)
- added ?: , , F.Cu at (35.0, 44.4)
- added ?: , , F.Cu at (122.7, 138.8)
- added ?: , , F.Cu at (122.7, 121.0)
- added ?: , , F.Cu at (35.1, 142.1)
- added ?: , , F.Cu at (122.7, 131.2)
- added ?: , , F.Cu at (46.2, 117.2)
- added ?: , , F.Cu at (111.0, 187.6)
- added ?: , , F.Cu at (172.0, 72.6)
- added ?: , , F.Cu at (122.5, 48.6)
- added ?: , , F.Cu at (259.5, 90.7)
- added ?: , , F.Cu at (172.0, 91.5)
- added ?: , , F.Cu at (117.6, 81.9)
- added ?: , , F.Cu at (197.1, 96.6)
- added ?: , , F.Cu at (58.2, 167.2)
- added ?: , , F.Cu at (234.0, 100.8)
- added ?: , , F.Cu at (111.0, 168.3)
- added ?: , , F.Cu at (97.2, 123.5)
- added ?: , , F.Cu at (242.7, 113.1)
- added ?: , , F.Cu at (234.0, 98.3)
- added ?: , , F.Cu at (45.9, 74.5)
- added ?: , , F.Cu at (122.5, 41.0)
- added ?: , , F.Cu at (100.7, 88.9)
- added ?: , , F.Cu at (182.9, 128.2)
- added ?: , , F.Cu at (35.0, 35.5)
- added ?: , , F.Cu at (45.9, 55.5)
- added ?: , , F.Cu at (97.2, 126.1)
- added ?: , , F.Cu at (58.2, 173.8)
- added ?: , , F.Cu at (108.4, 94.9)
- added ?: , , F.Cu at (122.7, 115.9)
- added ?: , , F.Cu at (172.0, 110.5)
- added ?: , , F.Cu at (46.0, 155.2)
- added ?: , , F.Cu at (259.5, 83.0)
- added ?: , , F.Cu at (122.7, 123.5)
- added ?: , , F.Cu at (118.5, 158.7)
- added ?: , , F.Cu at (237.6, 113.1)
- added ?: , , F.Cu at (255.4, 113.1)
- added ?: , , F.Cu at (60.3, 30.5)
- added ?: , , F.Cu at (97.2, 151.5)
- added ?: , , F.Cu at (46.0, 167.2)
- added ?: , , F.Cu at (35.0, 63.4)
- added ?: , , F.Cu at (58.1, 55.5)
- added ?: , , F.Cu at (60.1, 49.5)
- added ?: , , F.Cu at (97.0, 33.4)
- added ?: , , F.Cu at (182.9, 109.6)
- added ?: , , F.Cu at (35.1, 118.2)
- added ?: , , F.Cu at (97.2, 133.7)
- added ?: , , F.Cu at (46.0, 185.8)
- added ?: , , F.Cu at (195.1, 109.6)
- added ?: , , F.Cu at (197.1, 134.2)
- added ?: , , F.Cu at (58.4, 117.2)
- added ?: , , F.Cu at (122.5, 23.2)
- added ?: , , F.Cu at (183.1, 83.6)
- added ?: , , F.Cu at (122.7, 133.7)
- added ?: , , F.Cu at (45.9, 62.5)
- added ?: , , F.Cu at (105.8, 94.9)
- added ?: , , F.Cu at (97.0, 48.6)
- added ?: , , F.Cu at (60.1, 68.5)
- added ?: , , F.Cu at (233.9, 136.0)
- added ?: , , F.Cu at (35.0, 30.5)
- added ?: , , F.Cu at (103.2, 66.0)
- added ?: , , F.Cu at (117.7, 174.6)
- added ?: , , F.Cu at (259.5, 88.1)
- added ?: , , F.Cu at (58.2, 136.2)
- added ?: , , F.Cu at (97.2, 138.8)
- added ?: , , F.Cu at (113.4, 158.7)
- added ?: , , F.Cu at (234.0, 70.3)
- added D1: led smd 1206, LED_SMD:LED_1206_3216Metric, B.Cu at (76.0, 84.9)
- added D1: led smd 1206, LED_SMD:LED_1206_3216Metric, B.Cu at (212.9, 132.0)
- added D1: led smd 1206, LED_SMD:LED_1206_3216Metric, B.Cu at (76.1, 177.6)
- added D2: SM4007, Diode_SMD:D_MELF, B.Cu at (202.1, 134.4)
- added D2: SM4007, Diode_SMD:D_MELF, B.Cu at (65.2, 180.0)
- added D2: SM4007, Diode_SMD:D_MELF, B.Cu at (65.2, 87.3)
- added D3: led smd 1206, LED_SMD:LED_1206_3216Metric, B.Cu at (213.4, 113.3)
- added D3: led smd 1206, LED_SMD:LED_1206_3216Metric, B.Cu at (76.5, 66.2)
- added D3: led smd 1206, LED_SMD:LED_1206_3216Metric, B.Cu at (76.6, 158.8)
- added D4: SM4007, Diode_SMD:D_MELF, B.Cu at (202.1, 115.6)
- added D4: SM4007, Diode_SMD:D_MELF, B.Cu at (65.2, 68.5)
- added D4: SM4007, Diode_SMD:D_MELF, B.Cu at (65.2, 161.2)
- added D5: led smd 1206, LED_SMD:LED_1206_3216Metric, B.Cu at (212.9, 94.3)
- added D5: led smd 1206, LED_SMD:LED_1206_3216Metric, B.Cu at (76.1, 139.8)
- added D5: led smd 1206, LED_SMD:LED_1206_3216Metric, B.Cu at (76.0, 47.1)
- added D6: SM4007, Diode_SMD:D_MELF, B.Cu at (202.1, 96.6)
- added D6: SM4007, Diode_SMD:D_MELF, B.Cu at (65.2, 142.2)
- added D6: SM4007, Diode_SMD:D_MELF, B.Cu at (65.2, 49.5)
- added D7: led smd 1206, LED_SMD:LED_1206_3216Metric, B.Cu at (75.5, 28.1)
- added D7: led smd 1206, LED_SMD:LED_1206_3216Metric, B.Cu at (212.5, 75.2)
- added D7: led smd 1206, LED_SMD:LED_1206_3216Metric, B.Cu at (75.6, 120.8)
- added D8: SM4007, Diode_SMD:D_MELF, B.Cu at (202.1, 77.6)
- added D8: SM4007, Diode_SMD:D_MELF, B.Cu at (65.2, 30.5)
- added D8: SM4007, Diode_SMD:D_MELF, B.Cu at (65.2, 123.2)
- added Q1: MMBT3904, Package_TO_SOT_SMD:SOT-23, B.Cu at (70.7, 125.6)
- added Q1: MMBT3904, Package_TO_SOT_SMD:SOT-23, B.Cu at (207.5, 80.0)
- added Q1: MMBT3904, Package_TO_SOT_SMD:SOT-23, B.Cu at (70.6, 32.9)
- added Q2: MMBT3904, Package_TO_SOT_SMD:SOT-23, B.Cu at (70.7, 144.6)
- added Q2: MMBT3904, Package_TO_SOT_SMD:SOT-23, B.Cu at (70.6, 51.9)
- added Q2: MMBT3904, Package_TO_SOT_SMD:SOT-23, B.Cu at (207.5, 99.0)
- added Q3: MMBT3904, Package_TO_SOT_SMD:SOT-23, B.Cu at (70.6, 89.7)
- added Q3: MMBT3904, Package_TO_SOT_SMD:SOT-23, B.Cu at (207.5, 136.8)
- added Q3: MMBT3904, Package_TO_SOT_SMD:SOT-23, B.Cu at (70.7, 182.4)
- added Q4: MMBT3904, Package_TO_SOT_SMD:SOT-23, B.Cu at (207.5, 118.0)
- added Q4: MMBT3904, Package_TO_SOT_SMD:SOT-23, B.Cu at (70.7, 163.6)
- added Q4: MMBT3904, Package_TO_SOT_SMD:SOT-23, B.Cu at (70.6, 70.9)
- added R1: 220, Resistor_SMD:R_0805_2012Metric, B.Cu at (92.2, 172.9)
- added R1: 220, Resistor_SMD:R_0805_2012Metric, B.Cu at (92.1, 80.2)
- added R1: 220, Resistor_SMD:R_0805_2012Metric, B.Cu at (229.1, 127.3)
- added R10: 220, Resistor_SMD:R_0805_2012Metric, B.Cu at (90.3, 24.7)
- added R10: 220, Resistor_SMD:R_0805_2012Metric, B.Cu at (90.4, 117.4)
- added R10: 220, Resistor_SMD:R_0805_2012Metric, B.Cu at (227.2, 71.9)
- added R11: 1k, Resistor_SMD:R_0805_2012Metric, B.Cu at (76.1, 124.6)
- added R11: 1k, Resistor_SMD:R_0805_2012Metric, B.Cu at (213.0, 79.1)
- added R11: 1k, Resistor_SMD:R_0805_2012Metric, B.Cu at (76.0, 31.9)
- added R12: 220, Resistor_SMD:R_0805_2012Metric, B.Cu at (70.7, 120.8)
- added R12: 220, Resistor_SMD:R_0805_2012Metric, B.Cu at (70.6, 28.1)
- added R12: 220, Resistor_SMD:R_0805_2012Metric, B.Cu at (207.5, 75.2)
- added R2: 1k, Resistor_SMD:R_0805_2012Metric, B.Cu at (76.6, 181.4)
- added R2: 1k, Resistor_SMD:R_0805_2012Metric, B.Cu at (76.5, 88.8)
- added R2: 1k, Resistor_SMD:R_0805_2012Metric, B.Cu at (213.4, 135.9)
- added R3: 220, Resistor_SMD:R_0805_2012Metric, B.Cu at (70.6, 84.9)
- added R3: 220, Resistor_SMD:R_0805_2012Metric, B.Cu at (70.7, 177.6)
- added R3: 220, Resistor_SMD:R_0805_2012Metric, B.Cu at (207.5, 132.0)
- added R4: 220, Resistor_SMD:R_0805_2012Metric, B.Cu at (91.4, 61.8)
- added R4: 220, Resistor_SMD:R_0805_2012Metric, B.Cu at (228.3, 108.9)
- added R4: 220, Resistor_SMD:R_0805_2012Metric, B.Cu at (91.5, 154.5)
- added R5: 1k, Resistor_SMD:R_0805_2012Metric, B.Cu at (213.4, 117.1)
- added R5: 1k, Resistor_SMD:R_0805_2012Metric, B.Cu at (76.6, 162.6)
- added R5: 1k, Resistor_SMD:R_0805_2012Metric, B.Cu at (76.5, 69.9)
- added R6: 220, Resistor_SMD:R_0805_2012Metric, B.Cu at (207.5, 113.2)
- added R6: 220, Resistor_SMD:R_0805_2012Metric, B.Cu at (70.6, 66.1)
- added R6: 220, Resistor_SMD:R_0805_2012Metric, B.Cu at (70.7, 158.8)
- added R7: 220, Resistor_SMD:R_0805_2012Metric, B.Cu at (91.3, 42.8)
- added R7: 220, Resistor_SMD:R_0805_2012Metric, B.Cu at (91.4, 135.5)
- added R7: 220, Resistor_SMD:R_0805_2012Metric, B.Cu at (228.2, 89.9)
- added R8: 1k, Resistor_SMD:R_0805_2012Metric, B.Cu at (76.1, 143.6)
- added R8: 1k, Resistor_SMD:R_0805_2012Metric, B.Cu at (213.0, 98.0)
- added R8: 1k, Resistor_SMD:R_0805_2012Metric, B.Cu at (76.0, 50.9)
- added R9: 220, Resistor_SMD:R_0805_2012Metric, B.Cu at (207.5, 94.3)
- added R9: 220, Resistor_SMD:R_0805_2012Metric, B.Cu at (70.7, 139.8)
- added R9: 220, Resistor_SMD:R_0805_2012Metric, B.Cu at (70.6, 47.1)
- added U1: PC817, PC817SMD:SOIC254P1000X400-4N, B.Cu at (224.0, 76.5)
- added U1: PC817, PC817SMD:SOIC254P1000X400-4N, B.Cu at (87.1, 122.0)
- added U1: PC817, PC817SMD:SOIC254P1000X400-4N, B.Cu at (87.0, 29.4)
- added U2: PC817, PC817SMD:SOIC254P1000X400-4N, B.Cu at (87.1, 141.1)
- added U2: PC817, PC817SMD:SOIC254P1000X400-4N, B.Cu at (224.0, 95.5)
- added U2: PC817, PC817SMD:SOIC254P1000X400-4N, B.Cu at (87.0, 48.4)
- added U3: PC817, PC817SMD:SOIC254P1000X400-4N, B.Cu at (224.8, 133.3)
- added U3: PC817, PC817SMD:SOIC254P1000X400-4N, B.Cu at (88.0, 178.9)
- added U3: PC817, PC817SMD:SOIC254P1000X400-4N, B.Cu at (87.9, 86.2)
- added U4: PC817, PC817SMD:SOIC254P1000X400-4N, B.Cu at (87.3, 160.1)
- added U4: PC817, PC817SMD:SOIC254P1000X400-4N, B.Cu at (224.1, 114.5)
- added U4: PC817, PC817SMD:SOIC254P1000X400-4N, B.Cu at (87.2, 67.4)
Routing:
- net VIN: track 814.4 -> 1221.5 mm
- net D2: track 92.8 -> 139.2 mm
- net D25: track 64.7 -> 97.1 mm
- net COM1: track 50.6 -> 75.9 mm
- net D32: track 50.5 -> 75.7 mm
- net COM4: track 50.4 -> 75.7 mm
- net COM2: track 50.3 -> 75.5 mm
- net COM3: track 50.2 -> 75.2 mm
- net RX0: track 48.4 -> 72.6 mm
- net D23: track 45.1 -> 67.7 mm
- net RX2: track 42.1 -> 63.2 mm
- net TX0: track 39.2 -> 58.8 mm
- net Net-(D2-A): track 38.8 -> 58.2 mm
- net Net-(D8-A): track 38.0 -> 57.1 mm
- net Net-(SW1A-B): track 38.0 -> 56.9 mm
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